File: pcb/230ac_19dc.kicad_sch (KiCad schematic)
At the start: 49 parts, among them J1 6160.0159, Q1 BSP135H6433XTMA1, Q2 C3M0065090D, U1 LM5023, U2 PC817, U3 750313417, U5 MAX6101

Commit message: Rev 1.1
Created PCB design, minor changes to schematic diagram
Parts:
- C15, C5: footprint Capacitor_THT:CP_Radial_D12.5mm_P7.50mm -> Capacitor_THT:CP_Radial_D4.0mm_P2.00mm
- C6: footprint Capacitor_SMD:C_1206_3216Metric -> Capacitor_THT:CP_Radial_D4.0mm_P2.00mm
- F1: footprint Fuse:Fuse_1210_3225Metric -> Fuse:Fuse_Littelfuse-NANO2-462
- H1: footprint (none) -> TestPoint:TestPoint_THTPad_D2.5mm_Drill1.2mm
- H2: value GND -> GND1; footprint (none) -> TestPoint:TestPoint_THTPad_D2.5mm_Drill1.2mm
Connections:
- net VS is gone; now on net Vs: R7.1
- net Vs: now reaches C2.1, C3.1, C4.1, D1.1 (+), R1.1, R3.1, R4.1, U3.3 (PR13)
- net at D1.3: now also L1.3; no longer L1.2
- net at D1.4: now also L1.2; no longer L1.3
- net at C10.1, R8.1, U1.5 (CS): no longer Q2.3 (S), R12.2, R8.2
- net at Q1.4 (D_2), R7.2: no longer Q1.2 (D_1)
- new net: Q2.3 (S), R12.2, R8.2
- no-connect marks 0 -> 1
Changed lines of the file:
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@@
 	)
 	(junction
-		(at 52.07 78.74)
-		(diameter 0)
-		(color 0 0 0 0)
-	)
-	(junction
 		(at 254 26.67)
 		(diameter 0)
@@
 	)
 	(junction
-		(at 143.51 133.35)
-		(diameter 0)
-		(color 0 0 0 0)
-	)
-	(junction
 		(at 113.03 43.18)
 		(diameter 0)
@@
 	)
 	(junction
-		(at 151.13 133.35)
-		(diameter 0)
-		(color 0 0 0 0)
-	)
-	(junction
 		(at 182.88 54.61)
 		(diameter 0)
 		(color 0 0 0 0)
 	)
+	(no_connect
+		(at 52.07 82.55)
+	)
 	(wire
 		(pts
@@
 	(wire
 		(pts
-			(xy 52.07 78.74) (xy 52.07 77.47)
+			(xy 125.73 25.4) (xy 138.43 25.4)
 		)
 		(stroke
@@
 	(wire
 		(pts
-			(xy 26.67 78.74) (xy 52.07 78.74)
+			(xy 149.86 38.1) (xy 149.86 43.18)
 		)
 		(stroke
@@
 	(wire
 		(pts
-			(xy 149.86 38.1) (xy 149.86 43.18)
+			(xy 224.79 156.21) (xy 241.3 156.21)
 		)
 		(stroke
@@
 	(wire
 		(pts
-			(xy 224.79 156.21) (xy 241.3 156.21)
+			(xy 26.67 77.47) (xy 26.67 87.63)
 		)
 		(stroke
@@
 	(wire
 		(pts
-			(xy 138.43 25.4) (xy 125.73 25.4)
-		)
-		(stroke
-			(width 0)
-			(type default)
-		)
-	)
-	(wire
-		(pts
 			(xy 138.43 30.48) (xy 138.43 25.4)
 		)
@@
 	(wire
 		(pts
-			(xy 54.61 38.1) (xy 54.61 40.64)
+			(xy 52.07 77.47) (xy 26.67 77.47)
 		)
 		(stroke
@@
 	(wire
 		(pts
-			(xy 170.18 36.83) (xy 170.18 43.18)
+			(xy 54.61 38.1) (xy 54.61 40.64)
 		)
 		(stroke
@@
 	(wire
 		(pts
-			(xy 113.03 110.49) (xy 113.03 118.11)
+			(xy 170.18 36.83) (xy 170.18 43.18)
 		)
 		(stroke
@@
 	(wire
 		(pts
-			(xy 123.19 128.27) (xy 172.72 128.27)
+			(xy 113.03 110.49) (xy 113.03 118.11)
 		)
 		(stroke
@@
 	(wire
 		(pts
-			(xy 135.89 90.17) (xy 139.7 90.17)
+			(xy 123.19 128.27) (xy 172.72 128.27)
 		)
 		(stroke
@@
 	(wire
 		(pts
-			(xy 52.07 78.74) (xy 52.07 82.55)
+			(xy 135.89 90.17) (xy 139.7 90.17)
 		)
 		(stroke
@@
 	(wire
 		(pts
-			(xy 143.51 133.35) (xy 151.13 133.35)
-		)
-		(stroke
-			(width 0)
-			(type default)
-		)
-	)
-	(wire
-		(pts
 			(xy 218.44 151.13) (xy 218.44 137.16)
 		)
@@
 	(wire
 		(pts
-			(xy 26.67 87.63) (xy 26.67 78.74)
-		)
-		(stroke
-			(width 0)
-			(type default)
-		)
-	)
-	(wire
-		(pts
 			(xy 153.67 45.72) (xy 182.88 45.72)
 		)
@@
 		)
 	)
+	(global_label "Vs"
+		(shape input)
+		(at 52.07 69.85 90)
+		(fields_autoplaced yes)
+		(effects
+			(font
+				(size 1.27 1.27)
+			)
+			(justify left)
+		)
+		(property "Intersheetrefs" "${INTERSHEET_REFS}"
+			(at 52.07 64.7481 90)
+			(effects
+				(font
+					(size 1.27 1.27)
+				)
+				(justify left)
+				(hide yes)
+			)
+		)
+	)
+	(global_label "Vs"
+		(shape input)
+		(at 116.84 25.4 90)
+		(fields_autoplaced yes)
+		(effects
+			(font
+				(size 1.27 1.27)
+			)
+			(justify left)
+		)
+		(property "Intersheetrefs" "${INTERSHEET_REFS}"
+			(at 116.84 20.2981 90)
+			(effects
+				(font
+					(size 1.27 1.27)
+				)
+				(justify left)
+				(hide yes)
+			)
+		)
+	)
 	(global_label "Opto_signal"
 		(shape input)
@@
 			)
 		)
-		(property "Footprint" "Fuse:Fuse_1210_3225Metric"
+		(property "Footprint" "Fuse:Fuse_Littelfuse-NANO2-462"
 			(at 38.1 23.622 90)
 			(effects
@@
 			)
 		)
-		(property "Footprint" ""
+		(property "Footprint" "TestPoint:TestPoint_THTPad_D2.5mm_Drill1.2mm"
 			(at 275.59 26.67 0)
 			(effects
@@
 			)
 		)
-		(property "Value" "GND"
+		(property "Value" "GND1"
 			(at 279.4 40.6399 90)
 			(effects
@@
 			)
 		)
-		(property "Footprint" ""
+		(property "Footprint" "TestPoint:TestPoint_THTPad_D2.5mm_Drill1.2mm"
 			(at 275.59 39.37 0)
 			(effects
@@
 		)
 		(property "Value" "16pF/100V"
-			(at 191.008 62.23 0)
+			(at 191.516 62.23 0)
 			(effects
 				(font
@@
 			)
 		)
-		(property "Footprint" "Capacitor_THT:CP_Radial_D12.5mm_P7.50mm"
+		(property "Footprint" "Capacitor_THT:CP_Radial_D4.0mm_P2.00mm"
 			(at 238.76 147.6248 0)
 			(effects
@@
 	)
 	(symbol
-		(lib_id "power:VS")
-		(at 52.07 69.85 0)
-		(unit 1)
-		(exclude_from_sim no)
-		(in_bom yes)
-		(on_board yes)
-		(dnp no)
-		(fields_autoplaced yes)
-		(property "Reference" "#PWR010"
-			(at 52.07 73.66 0)
-			(effects
-				(font
-					(size 1.27 1.27)
-				)
-				(hide yes)
-			)
-		)
-		(property "Value" "VS"
-			(at 52.07 64.77 0)
-			(effects
-				(font
-					(size 1.27 1.27)
-				)
-			)
-		)
-		(property "Footprint" ""
-			(at 52.07 69.85 0)
-			(effects
-				(font
-					(size 1.27 1.27)
-				)
-				(hide yes)
-			)
-		)
-		(property "Datasheet" ""
-			(at 52.07 69.85 0)
-			(effects
-				(font
-					(size 1.27 1.27)
-				)
-				(hide yes)
-			)
-		)
-		(property "Description" "Power symbol creates a global label with name \"VS\""
-			(at 52.07 69.85 0)
-			(effects
-				(font
-					(size 1.27 1.27)
-				)
-				(hide yes)
-			)
-		)
-		(pin "1"
-		)
-		(instances
-			(project "230ac_19dc"
-				(path "/03082fd0-0b41-415a-ba03-08d032e83393"
-					(reference "#PWR010")
-					(unit 1)
-				)
-			)
-		)
-	)
-	(symbol
 		(lib_id "Device:C")
 		(at 138.43 34.29 0)
@@
 			)
 		)
-		(property "Footprint" "Capacitor_SMD:C_1206_3216Metric"
+		(property "Footprint" "Capacitor_THT:CP_Radial_D4.0mm_P2.00mm"
 			(at 122.8852 97.79 0)
 			(effects
@@
 			)
 		)
-		(property "Footprint" "Capacitor_THT:CP_Radial_D12.5mm_P7.50mm"
+		(property "Footprint" "Capacitor_THT:CP_Radial_D4.0mm_P2.00mm"
 			(at 136.8552 97.79 0)
 			(effects

Commit message: Rev 1.2
Minor changes in schematic - capacitor symbols
Parts:
- C12, C13, C14, C2, C3, C5, C6: symbol Device:C -> Device:C_Polarized
- J1: footprint private:61600159 -> 61600159
- U3: footprint private:SMD_13417_WRE -> SMD_13417_WRE
Connections:
- net at C6.1, C7.1, D4.1 (K)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: now also Q1.2 (D_1); no longer Q1.3 (S)
- net at D1.3: now also L1.2; no longer L1.3
- net at D1.4: now also L1.3; no longer L1.2
Other:
- moved on the sheet: R7
Changed lines of the file:
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@@
 	)
 	(junction
+		(at 116.84 25.4)
+		(diameter 0)
+		(color 0 0 0 0)
+	)
+	(junction
 		(at 261.62 163.83)
 		(diameter 0)
@@
 	(wire
 		(pts
-			(xy 26.67 77.47) (xy 26.67 87.63)
+			(xy 26.67 74.93) (xy 26.67 87.63)
 		)
 		(stroke
@@
 	(wire
 		(pts
+			(xy 116.84 22.86) (xy 116.84 25.4)
+		)
+		(stroke
+			(width 0)
+			(type default)
+		)
+	)
+	(wire
+		(pts
 			(xy 95.25 106.68) (xy 113.03 106.68)
 		)
@@
 	(wire
 		(pts
-			(xy 52.07 77.47) (xy 26.67 77.47)
-		)
-		(stroke
-			(width 0)
-			(type default)
-		)
-	)
-	(wire
-		(pts
 			(xy 54.61 38.1) (xy 54.61 40.64)
 		)
@@
 	(wire
 		(pts
+			(xy 26.67 67.31) (xy 26.67 66.04)
+		)
+		(stroke
+			(width 0)
+			(type default)
+		)
+	)
+	(wire
+		(pts
 			(xy 125.73 30.48) (xy 125.73 25.4)
 		)
@@
 	(wire
 		(pts
-			(xy 125.73 25.4) (xy 113.03 25.4)
+			(xy 125.73 25.4) (xy 116.84 25.4)
 		)
 		(stroke
@@
 	(wire
 		(pts
+			(xy 116.84 25.4) (xy 113.03 25.4)
+		)
+		(stroke
+			(width 0)
+			(type default)
+		)
+	)
+	(wire
+		(pts
 			(xy 243.84 39.37) (xy 254 39.37)
 		)
@@
 	(global_label "Vs"
 		(shape input)
-		(at 52.07 69.85 90)
+		(at 26.67 66.04 90)
 		(fields_autoplaced yes)
 		(effects
@@
 		)
 		(property "Intersheetrefs" "${INTERSHEET_REFS}"
-			(at 52.07 64.7481 90)
+			(at 26.67 60.9381 90)
 			(effects
 				(font
@@
 	(global_label "Vs"
 		(shape input)
-		(at 116.84 25.4 90)
+		(at 116.84 22.86 90)
 		(fields_autoplaced yes)
 		(effects
@@
 		)
 		(property "Intersheetrefs" "${INTERSHEET_REFS}"
-			(at 116.84 20.2981 90)
+			(at 116.84 17.7581 90)
 			(effects
 				(font
@@
 	)
 	(symbol
-		(lib_id "Device:C")
+		(lib_id "Device:C_Polarized")
 		(at 243.84 33.02 0)
 		(unit 1)
@@
 			)
 		)
-		(property "Description" "Unpolarized capacitor"
+		(property "Description" "Polarized capacitor"
 			(at 243.84 33.02 0)
 			(effects
@@
 	)
 	(symbol
-		(lib_id "Device:C")
+		(lib_id "Device:C_Polarized")
 		(at 125.73 34.29 0)
 		(unit 1)
@@
 			)
 		)
-		(property "Description" "Unpolarized capacitor"
+		(property "Description" "Polarized capacitor"
 			(at 125.73 34.29 0)
 			(effects
@@
 	)
 	(symbol
-		(lib_id "Device:C")
+		(lib_id "Device:C_Polarized")
 		(at 265.43 33.02 0)
 		(unit 1)
@@
 			)
 		)
-		(property "Description" "Unpolarized capacitor"
+		(property "Description" "Polarized capacitor"
 			(at 265.43 33.02 0)
 			(effects
@@
 			)
 		)
-		(property "Footprint" "private:61600159"
+		(property "Footprint" "61600159"
 			(at 11.43 -59.36 0)
 			(effects
@@
 	)
 	(symbol
-		(lib_id "Device:C")
+		(lib_id "Device:C_Polarized")
 		(at 138.43 34.29 0)
 		(unit 1)
@@
 			)
 		)
-		(property "Description" "Unpolarized capacitor"
+		(property "Description" "Polarized capacitor"
 			(at 138.43 34.29 0)
 			(effects
@@
 	)
 	(symbol
-		(lib_id "Device:C")
+		(lib_id "Device:C_Polarized")
 		(at 254 33.02 0)
 		(unit 1)
@@
 			)
 		)
-		(property "Description" "Unpolarized capacitor"
+		(property "Description" "Polarized capacitor"
 			(at 254 33.02 0)
 			(effects
@@
 	)
 	(symbol
-		(lib_name "750313417_1")
 		(lib_id "2024-11-26_16-51-12:750313417")
 		(at 189.23 26.67 0)
@@
 			)
 		)
-		(property "Footprint" "private:SMD_13417_WRE"
+		(property "Footprint" "SMD_13417_WRE"
 			(at 186.182 17.272 0)
 			(effects
@@
 	)
 	(symbol
-		(lib_id "Device:C")
+		(lib_id "Device:C_Polarized")
 		(at 121.92 93.98 0)
 		(unit 1)
@@
 			)
 		)
-		(property "Description" "Unpolarized capacitor"
+		(property "Description" "Polarized capacitor"
 			(at 121.92 93.98 0)
 			(effects
@@
 	(symbol
 		(lib_id "Device:R")
-		(at 52.07 73.66 0)
+		(at 26.67 71.12 0)
 		(unit 1)
 		(exclude_from_sim no)
@@
 		(dnp no)
 		(property "Reference" "R7"
-			(at 54.61 72.3899 0)
+			(at 29.21 69.8499 0)
 			(effects
 				(font
@@
 		)
 		(property "Value" "10K"
-			(at 54.61 74.9299 0)
+			(at 29.21 72.3899 0)
 			(effects
 				(font
@@
 		)
 		(property "Footprint" "Resistor_SMD:R_0805_2012Metric"
-			(at 50.292 73.66 90)
+			(at 24.892 71.12 90)
 			(effects
 				(font
@@
 		)
 		(property "Datasheet" "~"
-			(at 52.07 73.66 0)
+			(at 26.67 71.12 0)
 			(effects
 				(font
@@
 		)
 		(property "Description" "Resistor"
-			(at 52.07 73.66 0)
+			(at 26.67 71.12 0)
 			(effects
 				(font
@@
 	)
 	(symbol
-		(lib_id "Device:C")
+		(lib_id "Device:C_Polarized")
 		(at 135.89 93.98 0)
 		(unit 1)
@@
 			)
 		)
-		(property "Description" "Unpolarized capacitor"
+		(property "Description" "Polarized capacitor"
 			(at 135.89 93.98 0)
 			(effects
